Commit message: added imu

File: f110-fall2018-skeletons/simulator/racecar-simulator/racecar_description/urdf/racecar.xacro (robot description, xacro)
@@ -170,4 +170,31 @@
     <axis xyz="0 0 1" />
   </joint>
+  <!--gazebo imu-->
+  <link name="imu_link">
+  <inertial>
+    <mass value="0.001"/>
+    <origin rpy="0 0 0" xyz="0 0 0"/>
+    <inertia ixx="0.0001" ixy="0" ixz="0" iyy="0.000001" iyz="0" izz="0.0001"/>
+  </inertial>
+  <visual>
+    <origin rpy="0 0 0" xyz="0 0 0"/>
+    <geometry>
+      <box size="0.01 0.01 0.01"/><!--<box size="0.001 0.001 0.001"/>-->
+    </geometry>
+  </visual>
+  <collision>
+    <origin rpy="0 0 0" xyz="0 0 0"/>
+    <geometry>
+      <box size=".001 .001 .001"/>
+      <material name="grey" />
+    </geometry>
+  </collision>
+</link>
+<joint name="imu_joint" type="fixed">
+    <axis xyz="0.0 0 1"/> <!-- 0 1 0 -->
+    <origin xyz="0.1 0 0.035"/>
+    <parent link="chassis"/>
+    <child link="imu_link"/>
+  </joint>
   <!-- zed camera -->
   <link name="zed_camera_link">

Commit message: More Tests

File: f110-fall2018-skeletons/simulator/racecar-simulator/racecar_description/urdf/racecar.xacro (robot description, xacro)
@@ -192,5 +192,5 @@
 </link>
 <joint name="imu_joint" type="fixed">
-    <axis xyz="0.0 0 1"/> <!-- 0 1 0 -->
+    <axis xyz="0 0 1"/> <!-- 0 1 0 -->
     <origin xyz="0.1 0 0.035"/>
     <parent link="chassis"/>
